File: pcb/GNDPAD.kicad_pcb (KiCad board)
At the start: 2 copper layers, 78 x 78 mm, 49 parts, among them SW1 SW_Push_45deg, SW10 SW_Push_45deg, SW11 SW_Push_45deg, SW12 SW_Push_45deg, SW13 SW_Push_45deg, SW14 SW_Push_45deg, SW15 SW_Push_45deg, SW16 SW_Push_45deg, SW2 SW_Push_45deg, SW3 SW_Push_45deg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

Commit message: added journal
Parts:
- D1, D10, D11, D12, D13, D14, D15, D16, D2, D3, D4, D5, D6, D7, D8, D9: footprint Diode_THT:D_DO-35_SOD27_P7.62mm_Horizontal -> ScottoKeebs_Components:Diode_SOD-123
- moved D10 3.43 mm to (82.0, 77.1)
- moved D11 3.43 mm to (101.1, 77.1)
- moved D12 3.43 mm to (120.1, 77.1)
- moved D9 3.43 mm to (63.0, 77.1)
- moved D1 3.43 mm to (81.8, 38.7)
- moved D2 3.43 mm to (98.4, 38.5)
- moved D3 3.43 mm to (101.1, 38.5)
- moved D4 3.43 mm to (119.9, 38.5)
- moved D5 3.43 mm to (63.0, 57.4)
- moved D6 3.43 mm to (82.0, 57.4)
- moved D7 3.43 mm to (101.1, 57.4)
- moved D8 3.43 mm to (120.1, 57.4)
- moved D13 3.43 mm to (63.0, 96.1)
- moved D14 3.43 mm to (82.0, 96.1)
- moved D15 3.43 mm to (101.1, 96.1)
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Routing:
- net r4: track 133.8 -> 142.4 mm, vias 0 -> 4
- net r2: track 89.0 -> 97.0 mm, vias 6 -> 10
- net r1: track 69.6 -> 77.2 mm, vias 2 -> 6
- net r3: track 115.5 -> 122.6 mm, vias 6 -> 10
- net Net-(D1-A): track 17.3 -> 19.9 mm, vias 0 -> 1
- net +5V: track 321.0 -> 323.4 mm
- net Net-(D2-A): track 14.8 -> 12.6 mm
