File: pcb/GNDPAD.kicad_sch (KiCad schematic)
At the start: 49 parts, among them SW1 SW_Push_45deg, SW10 SW_Push_45deg, SW11 SW_Push_45deg, SW12 SW_Push_45deg, SW13 SW_Push_45deg, SW14 SW_Push_45deg, SW15 SW_Push_45deg, SW16 SW_Push_45deg, SW2 SW_Push_45deg, SW3 SW_Push_45deg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

Commit message: added journal
Parts:
- D1, D10, D11, D12, D13, D14, D15, D16, D2, D3, D4, D5, D6, D7, D8, D9: footprint Diode_THT:D_DO-35_SOD27_P7.62mm_Horizontal -> ScottoKeebs_Components:Diode_SOD-123
Changed lines of the file:
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@@
 			)
 		)
-		(property "Footprint" "Diode_THT:D_DO-35_SOD27_P7.62mm_Horizontal"
+		(property "Footprint" "ScottoKeebs_Components:Diode_SOD-123"
 			(at 38.1 129.54 0)
 			(effects
@@
 			)
 		)
-		(property "Footprint" "Diode_THT:D_DO-35_SOD27_P7.62mm_Horizontal"
+		(property "Footprint" "ScottoKeebs_Components:Diode_SOD-123"
 			(at 54.61 129.54 0)
 			(effects
@@
 			)
 		)
-		(property "Footprint" "Diode_THT:D_DO-35_SOD27_P7.62mm_Horizontal"
+		(property "Footprint" "ScottoKeebs_Components:Diode_SOD-123"
 			(at 87.63 106.68 0)
 			(effects
@@
 			)
 		)
-		(property "Footprint" "Diode_THT:D_DO-35_SOD27_P7.62mm_Horizontal"
+		(property "Footprint" "ScottoKeebs_Components:Diode_SOD-123"
 			(at 38.1 62.23 0)
 			(effects
@@
 			)
 		)
-		(property "Footprint" "Diode_THT:D_DO-35_SOD27_P7.62mm_Horizontal"
+		(property "Footprint" "ScottoKeebs_Components:Diode_SOD-123"
 			(at 87.63 83.82 0)
 			(effects
@@
 			)
 		)
-		(property "Footprint" "Diode_THT:D_DO-35_SOD27_P7.62mm_Horizontal"
+		(property "Footprint" "ScottoKeebs_Components:Diode_SOD-123"
 			(at 87.63 129.54 0)
 			(effects
@@
 			)
 		)
-		(property "Footprint" "Diode_THT:D_DO-35_SOD27_P7.62mm_Horizontal"
+		(property "Footprint" "ScottoKeebs_Components:Diode_SOD-123"
 			(at 71.12 129.54 0)
 			(effects
@@
 			)
 		)
-		(property "Footprint" "Diode_THT:D_DO-35_SOD27_P7.62mm_Horizontal"
+		(property "Footprint" "ScottoKeebs_Components:Diode_SOD-123"
 			(at 87.63 62.23 0)
 			(effects
@@
 			)
 		)
-		(property "Footprint" "Diode_THT:D_DO-35_SOD27_P7.62mm_Horizontal"
+		(property "Footprint" "ScottoKeebs_Components:Diode_SOD-123"
 			(at 38.1 106.68 0)
 			(effects
@@
 			)
 		)
-		(property "Footprint" "Diode_THT:D_DO-35_SOD27_P7.62mm_Horizontal"
+		(property "Footprint" "ScottoKeebs_Components:Diode_SOD-123"
 			(at 54.61 106.68 0)
 			(effects
@@
 			)
 		)
-		(property "Footprint" "Diode_THT:D_DO-35_SOD27_P7.62mm_Horizontal"
+		(property "Footprint" "ScottoKeebs_Components:Diode_SOD-123"
 			(at 54.61 62.23 0)
 			(effects
@@
 			)
 		)
-		(property "Footprint" "Diode_THT:D_DO-35_SOD27_P7.62mm_Horizontal"
+		(property "Footprint" "ScottoKeebs_Components:Diode_SOD-123"
 			(at 71.12 62.23 0)
 			(effects
@@
 			)
 		)
-		(property "Footprint" "Diode_THT:D_DO-35_SOD27_P7.62mm_Horizontal"
+		(property "Footprint" "ScottoKeebs_Components:Diode_SOD-123"
 			(at 71.12 106.68 0)
 			(effects
@@
 			)
 		)
-		(property "Footprint" "Diode_THT:D_DO-35_SOD27_P7.62mm_Horizontal"
+		(property "Footprint" "ScottoKeebs_Components:Diode_SOD-123"
 			(at 71.12 83.82 0)
 			(effects
@@
 			)
 		)
-		(property "Footprint" "Diode_THT:D_DO-35_SOD27_P7.62mm_Horizontal"
+		(property "Footprint" "ScottoKeebs_Components:Diode_SOD-123"
 			(at 38.1 83.82 0)
 			(effects
@@
 			)
 		)
-		(property "Footprint" "Diode_THT:D_DO-35_SOD27_P7.62mm_Horizontal"
+		(property "Footprint" "ScottoKeebs_Components:Diode_SOD-123"
 			(at 54.61 83.82 0)
 			(effects
