File: src/wind16.kicad_pcb (KiCad board)
At the start: 2 copper layers, 78 x 78 mm, 49 parts, among them SW1 SW_Push_45deg, SW10 SW_Push_45deg, SW11 SW_Push_45deg, SW12 SW_Push_45deg, SW13 SW_Push_45deg, SW14 SW_Push_45deg, SW15 SW_Push_45deg, SW16 SW_Push_45deg, SW2 SW_Push_45deg, SW3 SW_Push_45deg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

Commit message: stuff 1.2
Parts:
- U1: footprint Seeed Studio XIAO Series Library:XIAO-RP2040-DIP -> Seeed XIAO:XIAO-RP2040-DIP

Commit message: loads of shit 1.3
Parts:
- added REF**: MountingHole_2.2mm_M2, MountingHole:MountingHole_2.2mm_M2, F.Cu at (80.6, 66.8)
- added REF**: MountingHole_2.2mm_M2, MountingHole:MountingHole_2.2mm_M2, F.Cu at (99.8, 47.6)
- added REF**: MountingHole_2.2mm_M2, MountingHole:MountingHole_2.2mm_M2, F.Cu at (118.8, 47.6)
- added REF**: MountingHole_2.2mm_M2, MountingHole:MountingHole_2.2mm_M2, F.Cu at (80.6, 85.8)
- added REF**: MountingHole_2.2mm_M2, MountingHole:MountingHole_2.2mm_M2, F.Cu at (118.8, 85.8)
- SW10, SW11, SW12, SW13, SW14, SW15, SW16, SW2, SW3, SW4, SW5, SW6, SW7, SW8, SW9: footprint Button_Switch_Keyboard:SW_Cherry_MX_1.00u_PCB -> ScottoKeebs_Hotswap:Hotswap_MX_1.00u
- moved D4 16.7 mm to (136.6, 38.2)
- moved D7 16.5 mm to (117.6, 57.0)
- moved D3 16.5 mm to (117.6, 38.2)
- moved D8 16.5 mm to (136.6, 57.2)
- moved D10 16.4 mm to (98.4, 76.2)
- moved D11 16.4 mm to (117.5, 76.2)
- moved D12 16.4 mm to (136.5, 76.2)
- moved D14 16.4 mm to (98.4, 95.2)
- moved D15 16.4 mm to (117.5, 95.2)
- moved D16 16.4 mm to (136.5, 95.2)
- moved D13 16.4 mm to (79.3, 95.2)
- moved D9 16.4 mm to (79.3, 76.2)
- moved D6 16.4 mm to (98.4, 57.2)
- moved D5 16.4 mm to (79.3, 57.2)
- moved SW11 5.76 mm to (109.2, 76.3)
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Routing:
- net +5V: track 323.4 -> 347.1 mm, vias 12 -> 27
- net Net-(D24-DOUT): track 19.8 -> 36.9 mm, vias 0 -> 2
- net GND: track 345.9 -> 362.4 mm, vias 21 -> 19
- net r4: track 142.4 -> 126.0 mm, vias 4 -> 0
- net c3: track 107.9 -> 92.3 mm, vias 1 -> 2
- net r2: track 97.0 -> 84.9 mm, vias 10 -> 7
- net Net-(D17-DOUT): track 39.2 -> 27.8 mm, vias 0 -> 2
- net r3: track 122.6 -> 111.5 mm, vias 10 -> 7
- net c2: track 71.6 -> 61.3 mm, vias 1 -> 0
- net Net-(D25-DOUT): track 38.1 -> 27.9 mm
- net Net-(D26-DOUT): track 37.4 -> 27.4 mm
- net Net-(D18-DOUT): track 38.1 -> 28.5 mm
- net Net-(D19-DOUT): track 36.4 -> 27.8 mm, vias 0 -> 2
- net r1: track 77.2 -> 85.3 mm, vias 6 -> 8
- net Net-(D2-A): track 12.6 -> 4.51 mm
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
Commit message: gerbers, jlc, small changes
Other:
- board text added: "16"
- board text added: "wind"
Changed lines of the file:
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@@
+		)
+	)
+	(gr_text "16"
+		(at 98.4 85.4 0)
+		(layer "B.SilkS")
+		(effects
+			(font
+				(face "SF Pro")
+				(size 15 15)
+				(thickness 0.3)
+				(bold yes)
+			)
+			(justify bottom mirror)
+		)
+		(render_cache "16" 0
+			(polygon
+				(pts
+					(xy 105.529448 82.85) (xy 105.529448 70.866224) (xy 105.590814 70.866224) (xy 109.368945 73.43627)
+					(xy 109.368945 70.68121) (xy 105.539523 68.019574) (xy 102.484045 68.019574) (xy 102.484045 82.85)
+				)
+			)
+			(polygon
+				(pts
+					(xy 93.188467 83.084473) (xy 94.074431 83.030011) (xy 94.893444 82.870954) (xy 95.655015 82.610947)
+					(xy 96.368763 82.244827) (xy 97.019212 81.775659) (xy 97.612316 81.196781) (xy 98.114739 80.535583)
+					(xy 98.546148 79.755767) (xy 98.90375 78.841058) (xy 99.148863 77.887133) (xy 99.304799 76.79154)
+					(xy 99.359873 75.534621) (xy 99.359873 75.513555) (xy 99.269387 73.907059) (xy 99.01386 72.525619)
+					(xy 98.611574 71.337002) (xy 98.025765 70.238095) (xy 97.314806 69.354435) (xy 96.474755 68.657964)
+					(xy 95.510665 68.149015) (xy 94.415435 67.835642) (xy 93.159158 67.726482) (xy 92.213206 67.785878)
+					(xy 91.356444 67.957868) (xy 90.57629 68.236645) (xy 89.846078 68.624846) (xy 89.215938 69.092714)
+					(xy 88.675775 69.642568) (xy 88.23177 70.26946) (xy 87.910419 70.945898) (xy 87.706742 71.681385)
+					(xy 87.686592 71.783967) (xy 90.769547 71.783967) (xy 90.799772 71.69146) (xy 91.021176 71.266817)
+					(xy 91.314514 70.904692) (xy 91.676064 70.607917) (xy 92.113188 70.37896) (xy 92.602843 70.238166)
+					(xy 93.182056 70.18845) (xy 93.870081 70.262521) (xy 94.447354 70.473649) (xy 94.937856 70.818597)
+					(xy 95.347283 71.271834) (xy 95.692879 71.830584) (xy 95.972836 72.512116) (xy 96.244141 73.614685)
+					(xy 96.381332 74.897147) (xy 96.397818 75.206725) (xy 96.402398 75.517219) (xy 95.930704 77.994757)
+					(xy 95.840423 78.698549) (xy 95.574414 79.324659) (xy 95.155413 79.858169) (xy 94.607213 80.271711)
+					(xy 93.96628 80.533334) (xy 93.242506 80.622505) (xy 92.519471 80.53358) (xy 91.878715 80.272627)
+					(xy 91.328208 79.860907) (xy 90.901438 79.330155) (xy 90.627784 78.706787) (xy 90.535074 78.005748)
+					(xy 90.535074 77.984682) (xy 90.625404 77.246327) (xy 90.886784 76.61448) (xy 91.301441 76.082814)
+					(xy 91.84391 75.682083) (xy 92.48058 75.432726) (xy 93.213197 75.346859) (xy 93.946994 75.433606)
+					(xy 94.597138 75.687578) (xy 95.153128 76.093311) (xy 95.574414 76.624555) (xy 95.839517 77.254696)
+					(xy 95.930704 77.984682) (xy 96.575505 77.984682) (xy 96.575505 75.464096) (xy 96.353854 75.464096)
+					(xy 95.990133 74.811544) (xy 95.486487 74.23128) (xy 94.866211 73.753519) (xy 94.111705 73.376735)
+					(xy 93.274813 73.142507) (xy 92.311941 73.060746) (xy 91.370561 73.133485) (xy 90.537048 73.342971)
+					(xy 89.793186 73.68265) (xy 89.122384 74.150582) (xy 88.561136 74.718193) (xy 88.100583 75.394487)
+					(xy 87.765252 76.142366) (xy 87.560249 76.963132) (xy 87.489671 77.872025) (xy 87.489671 77.893091)
+					(xy 87.57484 78.88567) (xy 87.822104 79.775261) (xy 88.227895 80.581289) (xy 88.777064 81.300107)
+					(xy 89.447394 81.909742) (xy 90.252057 82.416774) (xy 91.132235 82.781986) (xy 92.105194 83.006764)
+				)
+			)
+		)
+	)
+	(gr_text "wind"
+		(at 98.2 65.6 0)
+		(layer "B.SilkS")
+		(effects
+			(font
+				(face "SF Pro")
+				(size 20 20)
+				(thickness 0.3)
+				(bold yes)
+			)
+			(justify bottom mirror)
+		)
+		(render_cache "wind" 0
+			(polygon
+				(pts
+					(xy 124.857884 62.2) (xy 128.753558 47.50635) (xy 124.734542 47.50635) (xy 122.519259 58.403244)
+					(xy 122.437438 58.403244) (xy 119.839915 47.50635) (xy 116.011409 47.50635) (xy 113.400452 58.403244)
+					(xy 113.318631 58.403244) (xy 111.089915 47.50635) (xy 107.15272 47.50635) (xy 111.034961 62.2)
+					(xy 115.287228 62.2) (xy 117.939706 51.809909) (xy 118.021527 51.809909) (xy 120.660571 62.2)
+				)
+			)
+			(polygon
+				(pts
+					(xy 105.488205 62.2) (xy 105.488205 47.50635) (xy 101.502162 47.50635) (xy 101.502162 62.2)
+				)
+			)
+			(polygon
+				(pts
+					(xy 103.495184 45.552407) (xy 104.076629 45.482641) (xy 104.580464 45.280004) (xy 105.025365 44.940579)
+					(xy 105.37231 44.500976) (xy 105.575613 44.019933) (xy 105.644521 43.481228) (xy 105.57518 42.935474)
+					(xy 105.371493 42.453046) (xy 105.025365 42.016992) (xy 104.580812 41.680473) (xy 104.076958 41.47934)
+					(xy 103.495184 41.410048) (xy 102.91422 41.479309) (xy 102.410751 41.680411) (xy 101.966224 42.016992)
+					(xy 101.619361 42.453133) (xy 101.415303 42.935556) (xy 101.345847 43.481228) (xy 101.414869 44.019853)
+					(xy 101.618543 44.500889) (xy 101.966224 44.940579) (xy 102.411099 45.280067) (xy 102.914549 45.482673)
+				)
+			)
+			(polygon
+				(pts
+					(xy 98.8448 62.2) (xy 98.8448 47.50635) (xy 94.858757 47.50635) (xy 94.858757 49.882833) (xy 94.776935 49.882833)
+					(xy 94.329375 49.103016) (xy 93.767052 48.451289) (xy 93.08189 47.914235) (xy 92.303399 47.52473)
+					(xy 91.387716 47.280235) (xy 90.304849 47.193719) (xy 89.1089 47.294732) (xy 88.109993 47.579218)
+					(xy 87.271136 48.031984) (xy 86.565491 48.655512) (xy 86.010272 49.417646) (xy 85.599513 50.326711)
+					(xy 85.338455 51.411566) (xy 85.245358 52.708722) (xy 85.245358 62.2) (xy 89.231402 62.2) (xy 89.231402 53.503733)
+					(xy 89.316297 52.562965) (xy 89.548512 51.83304) (xy 89.909175 51.26769) (xy 90.412445 50.841376)
+					(xy 91.069612 50.573621) (xy 91.929064 50.476343) (xy 92.773837 50.581574) (xy 93.476342 50.883007)
+					(xy 94.056321 51.365819) (xy 94.496056 52.018736) (xy 94.76392 52.790164) (xy 94.858757 53.723551)
+					(xy 94.858757 62.2)
+				)
+			)
+			(polygon
+				(pts
+					(xy 72.795079 50.014724) (xy 73.26224 49.190005) (xy 73.855093 48.502861) (xy 74.568887 47.94692)
+					(xy 75.393823 47.533217) (xy 76.298456 47.280715) (xy 77.308687 47.193719) (xy 78.511236 47.300478)
+					(xy 79.561664 47.607427) (xy 80.488729 48.107187) (xy 81.294909 48.788094) (xy 81.980237 49.65274)
+					(xy 82.547696 50.729134) (xy 82.936204 51.89029) (xy 83.183897 53.248962) (xy 83.271876 54.83852)
+					(xy 83.271876 54.854396) (xy 83.185307 56.43518) (xy 82.941135 57.792361) (xy 82.557466 58.957676)
+					(xy 81.995614 60.038065) (xy 81.313151 60.907183) (xy 80.507047 61.593056) (xy 79.578165 62.096678)
+					(xy 78.52921 62.405414) (xy 77.33189 62.51263) (xy 76.301835 62.425376) (xy 75.397487 62.174354)
+					(xy 74.576518 61.76294) (xy 73.87219 61.216922) (xy 73.288956 60.540146) (xy 72.835379 59.729483)
+					(xy 72.753558 59.729483) (xy 72.753558 62.2) (xy 68.734542 62.2) (xy 68.734542 54.83852) (xy 72.740125 54.83852)
+					(xy 72.740125 54.854396) (xy 72.848186 56.141213) (xy 73.14801 57.180809) (xy 73.648869 58.066666)
+					(xy 74.289845 58.697557) (xy 75.075063 59.094773) (xy 75.989776 59.230006) (xy 76.925712 59.093697)
+					(xy 77.709245 58.697557) (xy 78.340841 58.066502) (xy 78.824214 57.180809) (xy 79.108567 56.142434)
+					(xy 79.211339 54.854396) (xy 79.211339 54.83852) (xy 79.106554 53.539906) (xy 78.818108 52.506001)
+					(xy 78.330456 51.626031) (xy 77.703139 51.002686) (xy 76.925178 50.61141) (xy 75.989776 50.476343)
+					(xy 75.076305 50.612083) (xy 74.297173 51.010013) (xy 73.659473 51.638242) (xy 73.155337 52.519434)
+					(xy 72.85023 53.55309) (xy 72.740125 54.83852) (xy 68.734542 54.83852) (xy 68.734542 42.426099)
+					(xy 72.795079 42.426099)
+				)
+			)
 		)
 	)

Commit message: gerbs
Routing:
- net +5V: track 347.1 -> 352.9 mm
- net Net-(D17-DOUT): track 27.8 -> 30.8 mm
- net Net-(D27-DOUT): track 27.5 -> 29.9 mm
- net Net-(D18-DOUT): track 28.5 -> 29.5 mm
- net Net-(D19-DOUT): track 27.8 -> 28.6 mm
- net Net-(D23-DOUT): track 14.4 -> 15.2 mm
- net Net-(D25-DOUT): track 27.9 -> 27.3 mm
